Commit message: Feat:  Launch file and required config files are added to visualize robot's movement and TF (by using rviz)

File: robot_description/urdf/Coint5_r2.urdf (robot description, URDF)
Before this commit: robot Coint_5r2, 7 links, 6 joints
Links:
- added link world
- link Joint1: mass None -> 1.0
- link Joint2: mass None -> 1.0
- link Joint3: mass None -> 1.0
- link Joint4: mass None -> 1.0
- link Joint5: mass None -> 1.0
- link Joint6: mass None -> 1.0
- link base_link: mass None -> 1.0
Joints:
- added joint fix_to_world: type fixed, parent world, child base_link, origin xyz=0 0 0 rpy=0 0 0
